File: ac-switch-board/ac-switch-board.sch (KiCad schematic (older format))
At the start: 19 parts

Commit message: Updated board, added datasheets
Parts:
- removed F?: Fuse, symbol Fuse
- added C1, C10: 10uF, Capacitors_SMD:CP_Elec_4x4.5, symbol CP1
- added C15: 0.33uF, Capacitors_SMD:C_0805_HandSoldering, symbol C
- added C16: 0.1uF, Capacitors_SMD:C_0805_HandSoldering, symbol C
- added C17, C18, C3, C8: 100nF, Capacitors_SMD:C_1206_HandSoldering, symbol C
- added C19, C20: 1nF, Capacitors_SMD:C_0805_HandSoldering, symbol C
- added C2, C4: 20pF, Capacitors_SMD:C_0603, symbol C
- added C6: 6800uF, Capacitors_THT:CP_Radial_D18.0mm_P7.50mm, symbol CP1
- added CON1: AVR-ISP-10, Connectors:IDC_Header_Straight_10pins, symbol AVR-ISP-10
- added D2, D3, D5: LED, LEDs:LED_0603_HandSoldering, symbol LED
- added D6, D7: LL4148, Diodes_SMD:D_MiniMELF, symbol D
- added F1, F2: Fuse, Fuse_Holders_and_Fuses:Fuseholder5x20_horiz_SemiClosed_Casing10x25mm, symbol Fuse
- added J2: DIGITS, Pin_Headers:Pin_Header_Straight_1x08_Pitch2.54mm, symbol Conn_01x08
- added J3: SEGMENTS, Pin_Headers:Pin_Header_Straight_1x08_Pitch2.54mm, symbol Conn_01x08
- added J4: DISP0_EXTRAS, Pin_Headers:Pin_Header_Straight_1x04_Pitch2.54mm, symbol Conn_01x04
- added J5: DISP1_EXTRAS, Pin_Headers:Pin_Header_Straight_1x04_Pitch2.54mm, symbol Conn_01x04
- added J6: BLUEFRUIT_CONNECTOR, Pin_Headers:Pin_Header_Straight_1x09_Pitch2.54mm, symbol Conn_01x09_Female
- added J7: CH0_AC, Connectors:AK300-3, symbol Screw_Terminal_01x03
- added J8: CH1_AC, Connectors:AK300-3, symbol Screw_Terminal_01x03
- added K1: SRD_CH0, Relays_THT:Relay_SPDT_SANYOU_SRD_Series_Form_C, symbol SANYOU_SRD_Form_C
- added K2: SRD_CH1, Relays_THT:Relay_SPDT_SANYOU_SRD_Series_Form_C, symbol SANYOU_SRD_Form_C
- added LS1, LS2: Speaker, Pin_Headers:Pin_Header_Straight_1x02_Pitch2.54mm, symbol Speaker
- added Q1, Q2: S8050, TO_SOT_Packages_THT:TO-92_Molded_Narrow, symbol S8050
- added Q3, Q4: 2N7000, TO_SOT_Packages_THT:TO-92_Molded_Narrow, symbol 2N7000
- added R1, R15, R17, R2: 10k, Resistors_SMD:R_0805_HandSoldering, symbol R
- added R10, R9: 1.2k, Resistors_SMD:R_0805_HandSoldering, symbol R
- added R13: 1.37k, Resistors_SMD:R_0805_HandSoldering, symbol R
- added R14, R16: 100, Resistors_THT:R_Axial_DIN0207_L6.3mm_D2.5mm_P10.16mm_Horizontal, symbol R
- added R6, R7: 1k, Resistors_SMD:R_0805_HandSoldering, symbol R
- added U1: ATMEGA328P-PU, Housings_DIP:DIP-28_W7.62mm_Socket, symbol ATMEGA328P-PU
- added U2: MAX7221, Housings_DIP:DIP-24_W7.62mm_Socket, symbol MAX7221
- added U4, U5: PC817, Housings_DIP:DIP-4_W7.62mm, symbol PC817
- added U6: L7812, TO_SOT_Packages_THT:TO-220_Vertical, symbol L7812
- added U7, U8: ACS723, footprints:SOIC-8-N, symbol ACS723
- added Y1: 16MHz, Crystals:Crystal_HC49-4H_Vertical, symbol Crystal
- C11: renamed from C?; value C -> 0.015uf; footprint (none) -> Capacitors_SMD:C_0805_HandSoldering
- C12, C13: renamed from C?; footprint (none) -> Capacitors_SMD:C_0805_HandSoldering
- C14, C7, C9: renamed from C?; footprint (none) -> Capacitors_SMD:C_1206_HandSoldering
- C5: renamed from C?; value 2.2mF -> 6800uF; footprint (none) -> Capacitors_THT:CP_Radial_D18.0mm_P7.50mm
- D1: renamed from D?; value D_Bridge_+-AA -> 110B2 (W01G); footprint (none) -> Diodes_THT:Diode_Bridge_Round_D8.9mm; symbol D_Bridge_+-AA -> D_Bridge_+A-A
- D4: renamed from D?; footprint (none) -> footprints:D_SMA
- J1: renamed from J?; value Screw_Terminal_01x02 -> AC_IN; footprint (none) -> Connectors:AK300-3; symbol Screw_Terminal_01x02 -> Screw_Terminal_01x03
- L1: renamed from L?; footprint (none) -> footprints:L_Sumida_4.9x4.9mm_diag
- R11, R12, R3, R4, R5, R8: renamed from R?; footprint (none) -> Resistors_SMD:R_0805_HandSoldering
- U3: renamed from U?; footprint (none) -> footprints:SOIC-8-N
Connections:
- net GND: now also D1.3 (-), J1.2 (Pin_2), C1.2, C10.2, C15.2, C16.2, C17.2, C18.2, C19.2, C2.2, C20.2, C3.2, C4.2, C6.2, C8.2, D5.1 (K), J6.3 (Pin_3), Q1.1 (E), Q2.1 (E), Q3.1 (S), Q4.1 (S), R15.2, R17.2, U1.22 (GND), U1.8 (GND), U2.4 (GND), U2.9 (GND), U6.2 (GND), U7.5 (GND), U8.5 (GND); no longer D1.2 (-)
- net AC_IN_HOT: now reaches D1.4, J1.1 (Pin_1)
- net 15V renamed +15V
- net +15V: now also C15.1, C6.1, U6.1 (IN)
- net 5V renamed +5V
- net +5V: now also C1.1, C10.1, C17.1, C18.1, C3.1, C8.1, CON1.2, J4.1 (Pin_1), J4.2 (Pin_2), J5.1 (Pin_1), J5.2 (Pin_2), J6.4 (Pin_4), R1.1, R13.1, R14.1, R16.1, R2.1, R6.1, R7.1, U1.20 (AVCC), U1.7 (VCC), U2.19 (V+), U7.8 (VCC), U8.8 (VCC)
- new net: LS1.2, Q3.3 (D)
- new net: LS1.1, R14.2
- new net: LS2.2, Q4.3 (D)
- new net: LS2.1, R16.2
- new net: C19.1, U7.6 (BW_SEL)
- new net: F1.1, K1.1
- new net: F1.2, J7.1 (Pin_1)
- new net: C20.1, U8.6 (BW_SEL)
- new net: R2.2, U2.18 (ISET)
- new net: D6.2 (A), K1.2, Q1.3 (C)
- new net: R6.2, U4.1
- new net: D2.2 (A), U4.2
- new net: R9.1, U4.3
- new net: Q1.2 (B), R9.2
- new net: F2.1, K2.1
- new net: F2.2, J8.3 (Pin_3)
- new net: D7.2 (A), K2.2, Q2.3 (C)
- new net: R7.2, U5.1
- new net: D3.2 (A), U5.2
- new net: R10.1, U5.3
- new net: Q2.2 (B), R10.2
- new net: CON1.10, CON1.4, CON1.6, CON1.8
- new net: D5.2 (A), R13.2
- new net 12V: C16.1, U6.3 (OUT)
- new net AC_IN_NEUT: D1.2, J1.3 (Pin_3)
- new net AUD1: Q3.2 (G), R15.1, U1.5 ((PCINT19/OC2B/INT1)PD3)
- new net AUD2: Q4.2 (G), R17.1, U1.11 ((PCINT21/OC0B/T1)PD5)
- new net BLUEFRUIT_RST: J6.2 (Pin_2), U1.6 ((PCINT20/XCK/T0)PD4)
- new net BLUEFRUIT_SS: J6.9 (Pin_9), U1.15 ((PCINT1/OC1A)PB1)
- new net CH0_AC_MID: K1.3, U7.3 (IP-), U7.4 (IP-)
- new net CH0_AC_OUT: J7.3 (Pin_3), U7.1 (IP+), U7.2 (IP+)
- new net CH0_EN: D2.1 (K), U1.12 ((PCINT22/OC0A/AIN0)PD6)
- new net CH0_VIOUT: U1.27 ((PCINT12/SDA/ADC4)PC4), U7.7 (VIOUT)
- new net CH1_AC_MID: K2.3, U8.3 (IP-), U8.4 (IP-)
- new net CH1_AC_OUT: J8.1 (Pin_1), U8.1 (IP+), U8.2 (IP+)
- new net CH1_EN: D3.1 (K), U1.13 ((PCINT23/AIN1)PD7)
- new net CH1_VIOUT: U1.28 ((PCINT13/SCL/ADC5)PC5), U8.7 (VIOUT)
- new net DFU: J6.1 (Pin_1)
- new net DIG0: J2.1 (Pin_1), U2.2 (DIG_0)
- new net DIG1: J2.2 (Pin_2), U2.11 (DIG_1)
- new net DIG2: J2.3 (Pin_3), U2.6 (DIG_2)
- new net DIG3: J2.4 (Pin_4), U2.7 (DIG_3)
- new net DIG4: J2.5 (Pin_5), U2.3 (DIG_4)
- new net DIG5: J2.6 (Pin_6), U2.10 (DIG_5)
- new net DIG6: J2.7 (Pin_7), U2.5 (DIG_6)
- new net DIG7: J2.8 (Pin_8), U2.8 (DIG_7)
- new net DISPLAY_SS: U1.16 ((PCINT2/OC1B/~SS~)PB2), U2.12 (LOAD_(CS))
- new net DISP_COLON_0: J4.4 (Pin_4), U1.23 ((PCINT8/ADC0)PC0)
- new net DISP_COLON_1: J5.4 (Pin_4), U1.24 ((PCINT9/ADC1)PC1)
- new net DISP_EXTRA_0: J4.3 (Pin_3), U1.25 ((PCINT10/ADC2)PC2)
- new net DISP_EXTRA_1: J5.3 (Pin_3), U1.14 ((PCINT0/CLKO/ICP1)PB0)
- new net IRQ: J6.5 (Pin_5), U1.4 ((PCINT18/INT0)PD2)
- new net MISO: CON1.9, J6.7 (Pin_7), U1.18 ((PCINT4/MISO)PB4)
- new net MOSI: CON1.1, J6.8 (Pin_8), U1.17 ((PCINT3/OC2A/MOSI)PB3), U2.1 (DIN)
- new net RESET: CON1.5, R1.2, U1.1 ((PCINT14/~RESET~)PC6)
- new net SCK: CON1.7, J6.6 (Pin_6), U1.19 ((PCINT5/SCK)PB5), U2.13 (CLK)
- new net SEGA: J3.3 (Pin_3), U2.14 (SEG_A)
- new net SEGB: J3.1 (Pin_1), U2.16 (SEG_B)
- new net SEGC: J3.4 (Pin_4), U2.20 (SEG_C)
- new net SEGD: J3.8 (Pin_8), U2.23 (SEG_D)
- new net SEGDP: J3.6 (Pin_6), U2.22 (SEG_DP)
- new net SEGE: J3.7 (Pin_7), U2.21 (SEG_E)
- new net SEGF: J3.5 (Pin_5), U2.15 (SEG_F)
- new net SEGG: J3.2 (Pin_2), U2.17 (SEG_G)
- new net VCOIL: D6.1 (K), D7.1 (K), K1.5, K2.5, U4.4, U5.4
- new net XTAL1: C2.1, U1.9 ((PCINT6/XTAL1/TOSC1)PB6), Y1.2
- new net XTAL2: C4.1, U1.10 ((PCINT7/XTAL2/TOSC2)PB7), Y1.1
- no-connect marks 0 -> 11
Other:
- note added: "03/02/2018\n"
- note added: "1.0\n"
- note added: "120 VAC to 15VDC Rectifier"
- note added: "Bluetooth Controlled AC Switch"
- note added: "DC 15V to 12V, 5V Power Supply\n"
- note added: "Display System"
- note added: "Microcontroller Processing (ATMega)"
- note added: "Microcontroller Processing (Bluetooth)\n"
- note added: "Sound\nSystem"
- moved on the sheet: C11, C12, C13, C14, C5, C7, C9, D1, D4, L1, R11, R12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
