File: ac-switch-board-minimal/ac-switch-board-minimal.sch (KiCad schematic (older format))
At the start: 60 parts, among them CON1 AVR-ISP-10, J1 AC_IN, J10 BACKUP_VOUT, J11 BACKUP_VIN, J12 CH0_AC, J13 CH1_AC, J2 DIGITS, J3 SEGMENTS, J4 DISP0_EXTRAS, J5 DISP1_EXTRAS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

Commit message: board progress
Parts:
- removed CON1: AVR-ISP-10, Connectors:IDC_Header_Straight_10pins, symbol AVR-ISP-10
- added CON1: AVR-ISP-6, Connectors:IDC_Header_Straight_6pins, symbol AVR-ISP-6
- added J14: UART, Pin_Headers:Pin_Header_Straight_1x02_Pitch2.54mm, symbol Conn_01x02
- added J15: Conn_01x01, Pin_Headers:Pin_Header_Straight_1x01_Pitch2.54mm, symbol Conn_01x01
- added J16: SEGMENTS1, Pin_Headers:Pin_Header_Straight_1x08_Pitch2.54mm, symbol Conn_01x08
- J3: value SEGMENTS -> SEGMENTS0
- R11, R9: footprint Resistors_THT:R_Axial_DIN0207_L6.3mm_D2.5mm_P10.16mm_Horizontal -> Resistors_THT:R_Axial_DIN0207_L6.3mm_D2.5mm_P5.08mm_Vertical
Connections:
- net +5V: now also CON1.2
- net GND: now also CON1.6
- net MISO: now also CON1.4
- net MOSI: now also CON1.1
- net RESET: now also CON1.5
- net SCK: now also CON1.3
- net SEGA: now also J16.3 (Pin_3)
- net SEGB: now also J16.1 (Pin_1)
- net SEGC: now also J16.4 (Pin_4)
- net SEGD: now also J16.8 (Pin_8)
- net SEGDP: now also J16.6 (Pin_6)
- net SEGE: now also J16.7 (Pin_7)
- net SEGF: now also J16.5 (Pin_5)
- net SEGG: now also J16.2 (Pin_2)
- net at U1.2 ((PCINT16/RXD)PD0): now also J14.1 (Pin_1)
- net at U1.26 ((PCINT11/ADC3)PC3): now also J15.1 (Pin_1)
- net at U1.3 ((PCINT17/TXD)PD1): now also J14.2 (Pin_2)
- no-connect marks 7 -> 3
Other:
- moved on the sheet: C10, C8, J2, J3, J4, J5, R2, U2

Commit message: More small board tweaks
Parts:
- added D4: LED, Pin_Headers:Pin_Header_Straight_1x02_Pitch2.54mm, symbol LED
- added R13: 220, Resistors_SMD:R_0805_HandSoldering, symbol R
Connections:
- net +5V: now also R13.1
- net GND: now also D4.1 (K)
- new net: D4.2 (A), R13.2
Changed lines of the file:
@@
 F 1 "ATMEGA328P-PU" H 2450 2150 50  0000 L BNN
 F 2 "Housings_DIP:DIP-28_W7.62mm_Socket" H 2050 3550 50  0001 C CIN
-F 3 "" H 2050 3550 50  0001 C CNN
+F 3 "http://ww1.microchip.com/downloads/en/DeviceDoc/Atmel-42735-8-bit-AVR-Microcontroller-ATmega328-328P_Datasheet.pdf" H 2050 3550 50  0001 C CNN
 	1    2050 3550
 	1    0    0    -1
@@
 F 1 "2N7000" H 9600 1850 50  0000 L CNN
 F 2 "TO_SOT_Packages_THT:TO-92_Molded_Narrow" H 9600 1775 50  0001 L CIN
-F 3 "" H 9400 1850 50  0001 L CNN
+F 3 "https://www.digikey.com/product-detail/en/fairchild-on-semiconductor/2N7000/2N7000FS-ND/244278" H 9400 1850 50  0001 L CNN
 	1    9400 1850
 	1    0    0    -1
@@
 F 1 "2N7000" H 10750 1850 50  0000 L CNN
 F 2 "TO_SOT_Packages_THT:TO-92_Molded_Narrow" H 10750 1775 50  0001 L CIN
-F 3 "" H 10550 1850 50  0001 L CNN
+F 3 "https://www.digikey.com/product-detail/en/fairchild-on-semiconductor/2N7000/2N7000FS-ND/244278" H 10550 1850 50  0001 L CNN
 	1    10550 1850
 	1    0    0    -1
@@
 F 1 "BLUEFRUIT_CONNECTOR" H 5300 6650 50  0000 C CNN
 F 2 "Pin_Headers:Pin_Header_Straight_1x09_Pitch2.54mm" H 5300 7150 50  0001 C CNN
-F 3 "" H 5300 7150 50  0001 C CNN
+F 3 "https://www.adafruit.com/product/2633" H 5300 7150 50  0001 C CNN
 	1    5300 7150
 	-1   0    0    1
@@
 Text Label 950  7500 0    60   ~ 0
 SEGD
+$Comp
+L R R13
+U 1 1 5A8284E6
+P 8200 1050
+F 0 "R13" V 8280 1050 50  0000 C CNN
+F 1 "220" V 8200 1050 50  0000 C CNN
+F 2 "Resistors_SMD:R_0805_HandSoldering" V 8130 1050 50  0001 C CNN
+F 3 "" H 8200 1050 50  0001 C CNN
+	1    8200 1050
+	1    0    0    -1
+$EndComp
+$Comp
+L LED D4
+U 1 1 5A82857F
+P 8200 1450
+F 0 "D4" H 8200 1550 50  0000 C CNN
+F 1 "LED" H 8200 1350 50  0000 C CNN
+F 2 "Pin_Headers:Pin_Header_Straight_1x02_Pitch2.54mm" H 8200 1450 50  0001 C CNN
+F 3 "" H 8200 1450 50  0001 C CNN
+	1    8200 1450
+	0    -1   -1   0
+$EndComp
+Wire Wire Line
+	8200 1300 8200 1200
+$Comp
+L +5V #PWR051
+U 1 1 5A82872B
+P 8200 900
+F 0 "#PWR051" H 8200 750 50  0001 C CNN
+F 1 "+5V" H 8200 1040 50  0000 C CNN
+F 2 "" H 8200 900 50  0001 C CNN
+F 3 "" H 8200 900 50  0001 C CNN
+	1    8200 900
+	1    0    0    -1
+$EndComp
+$Comp
+L GND #PWR052
+U 1 1 5A8287C1
+P 8200 1600
+F 0 "#PWR052" H 8200 1350 50  0001 C CNN
+F 1 "GND" H 8200 1450 50  0000 C CNN
+F 2 "" H 8200 1600 50  0001 C CNN
+F 3 "" H 8200 1600 50  0001 C CNN
+	1    8200 1600
+	1    0    0    -1
+$EndComp
 $EndSCHEMATC

Commit message: Board work
Parts:
- J14: footprint Pin_Headers:Pin_Header_Straight_1x02_Pitch2.54mm -> Pin_Headers:Pin_Header_Straight_1x03_Pitch2.54mm; symbol Conn_01x02 -> Conn_01x03
Connections:
- net GND: now also J14.3 (Pin_3)
Changed lines of the file:
@@
 	9150 5250 8750 5250
 $Comp
-L Conn_01x02 J14
+L Conn_01x03 J14
 U 1 1 5A7D908B
-P 4000 4050
-F 0 "J14" H 4000 4150 50  0000 C CNN
-F 1 "UART" H 4000 3850 50  0000 C CNN
-F 2 "Pin_Headers:Pin_Header_Straight_1x02_Pitch2.54mm" H 4000 4050 50  0001 C CNN
-F 3 "" H 4000 4050 50  0001 C CNN
-	1    4000 4050
+P 4000 4150
+F 0 "J14" H 4000 4250 50  0000 C CNN
+F 1 "UART" H 4000 3950 50  0000 C CNN
+F 2 "Pin_Headers:Pin_Header_Straight_1x03_Pitch2.54mm" H 4000 4150 50  0001 C CNN
+F 3 "" H 4000 4150 50  0001 C CNN
+	1    4000 4150
 	1    0    0    -1
 $EndComp
@@
 	1    0    0    -1
 $EndComp
+$Comp
+L GND #PWR?
+U 1 1 5A8752EE
+P 3800 4250
+F 0 "#PWR?" H 3800 4000 50  0001 C CNN
+F 1 "GND" H 3800 4100 50  0000 C CNN
+F 2 "" H 3800 4250 50  0001 C CNN
+F 3 "" H 3800 4250 50  0001 C CNN
+	1    3800 4250
+	1    0    0    -1
+$EndComp

Commit message: Board things, including errata list for next version
Parts:
- added J17: XTRA_GND, Pin_Headers:Pin_Header_Straight_1x03_Pitch2.54mm, symbol Conn_01x03
- C1, C10: DigiKey (none) -> PCE3948CT-ND; MPN (none) -> EEE-1VA100WR
- C11: DigiKey (none) -> 490-1643-1-ND; MPN (none) -> GRM2195C1H153JA01D
- C12: DigiKey (none) -> 311-1121-1-ND; MPN (none) -> CC0805JRNPO9BN681
- C13: DigiKey (none) -> 311-1107-1-ND; MPN (none) -> CC0805JRNPO9BN470
- C14: DigiKey (none) -> 1276-6641-1-ND; MPN (none) -> CL31B106MOHNNNE
- C15, C16, C3, C8, C9: DigiKey (none) -> 399-1249-1-ND; MPN (none) -> C1206C104K5RAC7867
- C17, C18: DigiKey (none) -> 399-1147-1-ND; MPN (none) -> C0805C102K5RACTU
- C2: DigiKey (none) -> 1276-2220-1-ND; MPN (none) -> CL10C200JB8NCNC
- C5, C6: DigiKey (none) -> P15173-ND; MPN (none) -> EEU-HD1V682
- C7: DigiKey (none) -> 399-8153-1-ND; MPN (none) -> C1206C106M3PACTU
- D1: DigiKey (none) -> W01G-E4/51GI-ND; MPN (none) -> W01G-E4/51
- D2: DigiKey (none) -> B220A-FDICT-ND; MPN (none) -> B220A-13-F
- D3: DigiKey SML-D12V1WT86 -> SML-D12V1WT86CT-ND; MPN (none) -> SML-D12V1WT86
- L1: DigiKey (none) -> 308-2037-1-ND; MPN (none) -> CDRH4D28CLDNP-3R3PC
- R1, R10, R12, R2, R6: DigiKey (none) -> P10KDACT-ND; MPN (none) -> ERA-6AEB103V
- R13: DigiKey (none) -> RHM220KCT-ND; MPN (none) -> ESR10EZPJ221
- R3: DigiKey (none) -> RR12P150KDCT-ND; MPN (none) -> RR1220P-154-D
- R4: DigiKey (none) -> 311-48.7KCRCT-ND; MPN (none) -> RC0805FR-0748K7L
- R5: DigiKey (none) -> 311-17.4KCRCT-ND; MPN (none) -> RC0805FR-0717K4L
- R7: DigiKey (none) -> 311-1.87KCRCT-ND; MPN (none) -> RC0805FR-071K87L
- R8: DigiKey (none) -> 311-1.37KCRCT-ND; MPN (none) -> RC0805FR-071K37L
- U3: DigiKey (none) -> 296-39414-1-ND; MPN (none) -> TPS54232DR
- U4, U5: DigiKey (none) -> 620-1641-1-ND; MPN (none) -> ACS723LLCTR-05AB-T
Connections:
- net +5V: now also R2.2; no longer R2.1
- net GND: now also J17.1 (Pin_1), J17.2 (Pin_2), J17.3 (Pin_3)
- net at C9.1, U3.8 (PH): now also D2.1 (K), L1.1
- net at U2.18 (ISET): now also R2.1; no longer R2.2
