File: 7segboard/7segboard.kicad_pcb (KiCad board)
At the start: 2 copper layers, 19.7 x 41.3 mm, 8 parts, among them J1 SEGMENTS, J2 DIGITS, J3 EXTRAS, M1 M1, M2 M2

Commit message: board adds
Parts:
- moved J3 1.14 mm to (137.2, 123.8)
- moved J2 0.64 mm to (137.2, 103.5)
Routing:
- net /DIG3: track 22.1 -> 17.5 mm
- net /EXTRA: track 20.1 -> 22.0 mm
- net Net-(J3-Pad1): track 8.49 -> 9.84 mm
- net /DIG2: track 11.6 -> 12.4 mm
- net /COLON: track 6.37 -> 5.82 mm
Changed lines of the file:
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@@
     (thickness 1.6)
     (drawings 6)
-    (tracks 75)
+    (tracks 80)
     (zones 0)
     (modules 8)
@@
   )
   (module Pin_Headers:Pin_Header_Straight_1x04_Pitch2.54mm (layer B.Cu)
-    (at 137.16 104.14 180)
+    (at 137.16 103.505 180)
     (descr "Through hole straight pin header, 1x04, 2.54mm pitch, single row")
     (tags "Through hole pin header THT 1x04 2.54mm single row")
@@
   )
   (module Pin_Headers:Pin_Header_Straight_1x04_Pitch2.54mm (layer B.Cu)
-    (at 137.16 124.968)
+    (at 137.16 123.825)
     (descr "Through hole straight pin header, 1x04, 2.54mm pitch, single row")
     (tags "Through hole pin header THT 1x04 2.54mm single row")
@@
   (segment (start 143.51 112.395) (end 143.51 120.015) (width 0.25) (layer B.Cu) (net 8))
   (segment (start 141.6177 110.9091) (end 141.605 111.125) (width 0.25) (layer F.Cu) (net 8) (status 80000))
+  (segment (start 137.16 103.505) (end 139.2936 103.505) (width 0.25) (layer B.Cu) (net 9))
+  (segment (start 139.2936 103.505) (end 141.6177 105.8291) (width 0.25) (layer B.Cu) (net 9))
   (segment (start 141.6177 105.8291) (end 141.605 106.045) (width 0.25) (layer B.Cu) (net 9) (status 80000))
-  (segment (start 141.605 106.045) (end 139.7 104.14) (width 0.25) (layer B.Cu) (net 9) (status 80000))
-  (segment (start 139.7 104.14) (end 137.16 104.14) (width 0.25) (layer B.Cu) (net 9) (status 80000))
+  (segment (start 137.16 106.045) (end 139.2936 106.045) (width 0.25) (layer B.Cu) (net 10))
+  (segment (start 139.2936 106.045) (end 141.6177 108.3691) (width 0.25) (layer B.Cu) (net 10))
   (segment (start 141.6177 108.3691) (end 141.605 108.585) (width 0.25) (layer B.Cu) (net 10) (status 80000))
-  (segment (start 141.605 108.585) (end 139.7 106.68) (width 0.25) (layer B.Cu) (net 10) (status 80000))
-  (segment (start 139.7 106.68) (end 137.16 106.68) (width 0.25) (layer B.Cu) (net 10) (status 80000))
   (segment (start 141.6177 118.5291) (end 141.605 118.745) (width 0.25) (layer F.Cu) (net 11) (status 80000))
   (segment (start 141.605 118.745) (end 138.43 115.57) (width 0.25) (layer F.Cu) (net 11) (status 80000))
-  (segment (start 138.43 115.57) (end 138.43 110.49) (width 0.25) (layer F.Cu) (net 11) (status 80000))
-  (segment (start 138.43 110.49) (end 137.16 109.22) (width 0.25) (layer F.Cu) (net 11) (status 80000))
-  (segment (start 137.16 111.76) (end 135.89 113.03) (width 0.25) (layer F.Cu) (net 12) (status 80000))
-  (segment (start 135.89 113.03) (end 135.89 126.365) (width 0.25) (layer F.Cu) (net 12) (status 80000))
-  (segment (start 135.89 126.365) (end 139.065 126.365) (width 0.25) (layer F.Cu) (net 12) (status 80000))
-  (segment (start 139.065 126.365) (end 141.605 123.825) (width 0.25) (layer F.Cu) (net 12) (status 80000))
+  (segment (start 138.43 115.57) (end 138.43 109.855) (width 0.25) (layer F.Cu) (net 11) (status 80000))
+  (segment (start 138.43 109.855) (end 137.16 108.585) (width 0.25) (layer F.Cu) (net 11) (status 80000))
+  (segment (start 141.6177 118.5291) (end 141.605 118.745) (width 0.25) (layer F.Cu) (net 11) (status 80000))
+  (segment (start 137.16 111.125) (end 135.89 112.395) (width 0.25) (layer F.Cu) (net 12) (status 80000))
+  (segment (start 135.89 112.395) (end 135.89 117.475) (width 0.25) (layer F.Cu) (net 12) (status 80000))
+  (segment (start 135.89 117.475) (end 138.43 117.475) (width 0.25) (layer F.Cu) (net 12) (status 80000))
+  (segment (start 138.43 117.475) (end 140.335 119.38) (width 0.25) (layer F.Cu) (net 12) (status 80000))
+  (segment (start 140.335 119.38) (end 140.335 122.555) (width 0.25) (layer F.Cu) (net 12) (status 80000))
+  (segment (start 140.335 122.555) (end 141.605 123.825) (width 0.25) (layer F.Cu) (net 12) (status 80000))
   (segment (start 141.605 123.825) (end 141.6177 123.6091) (width 0.25) (layer F.Cu) (net 12) (status 80000))
-  (segment (start 137.16 124.968) (end 137.16 125.095) (width 0.25) (layer B.Cu) (net 13) (status 80000))
-  (segment (start 137.16 125.095) (end 142.875 130.81) (width 0.25) (layer B.Cu) (net 13) (status 80000))
+  (segment (start 141.605 123.825) (end 141.6177 123.6091) (width 0.25) (layer F.Cu) (net 12) (status 80000))
+  (segment (start 142.748 131.064) (end 142.748 129.413) (width 0.25) (layer B.Cu) (net 13))
+  (segment (start 142.748 129.413) (end 137.16 123.825) (width 0.25) (layer B.Cu) (net 13))
   (segment (start 142.875 130.81) (end 142.748 131.064) (width 0.25) (layer B.Cu) (net 13) (status 80000))
+  (segment (start 139.7 120.65) (end 139.7 119.38) (width 0.25) (layer B.Cu) (net 14))
+  (segment (start 139.065 118.745) (end 137.16 118.745) (width 0.25) (layer B.Cu) (net 14))
+  (segment (start 139.7 119.38) (end 139.065 118.745) (width 0.25) (layer B.Cu) (net 14))
+  (segment (start 139.7 121.92) (end 139.7 120.65) (width 0.25) (layer B.Cu) (net 14))
   (segment (start 151.765 121.285) (end 147.955 125.095) (width 0.25) (layer B.Cu) (net 14) (status 80000))
+  (segment (start 147.955 125.095) (end 140.335 125.095) (width 0.25) (layer B.Cu) (net 14) (status 80000))
+  (segment (start 139.7 124.46) (end 139.7 121.92) (width 0.25) (layer B.Cu) (net 14))
+  (segment (start 139.7 124.46) (end 140.335 125.095) (width 0.25) (layer B.Cu) (net 14))
   (segment (start 151.7777 121.0691) (end 151.765 121.285) (width 0.25) (layer B.Cu) (net 14) (status 80000))
-  (segment (start 139.7 124.46) (end 140.335 125.095) (width 0.25) (layer B.Cu) (net 14))
-  (segment (start 139.7 124.46) (end 139.7 121.92) (width 0.25) (layer B.Cu) (net 14))
-  (segment (start 147.955 125.095) (end 140.335 125.095) (width 0.25) (layer B.Cu) (net 14) (status 80000))
-  (segment (start 139.7 121.92) (end 137.795 120.015) (width 0.25) (layer B.Cu) (net 14) (status 80000))
-  (segment (start 137.795 120.015) (end 137.16 120.015) (width 0.25) (layer B.Cu) (net 14) (status 80000))
-  (segment (start 137.16 120.015) (end 137.16 119.888) (width 0.25) (layer B.Cu) (net 14) (status 80000))
+  (segment (start 141.6177 113.4491) (end 139.9159 113.4491) (width 0.25) (layer B.Cu) (net 15))
+  (segment (start 139.9159 113.4491) (end 137.16 116.205) (width 0.25) (layer B.Cu) (net 15))
   (segment (start 141.6177 113.4491) (end 141.605 113.665) (width 0.25) (layer B.Cu) (net 15) (status 80000))
-  (segment (start 141.605 113.665) (end 137.795 117.475) (width 0.25) (layer B.Cu) (net 15) (status 80000))
-  (segment (start 137.795 117.475) (end 137.16 117.475) (width 0.25) (layer B.Cu) (net 15) (status 80000))
-  (segment (start 137.16 117.475) (end 137.16 117.348) (width 0.25) (layer B.Cu) (net 15) (status 80000))
   (segment (start 151.7777 123.6091) (end 151.765 123.825) (width 0.25) (layer F.Cu) (net 16) (status 80000))
   (segment (start 151.765 123.825) (end 150.495 125.095) (width 0.25) (layer F.Cu) (net 16) (status 80000))
@@
   (segment (start 150.495 114.935) (end 151.765 116.205) (width 0.25) (layer F.Cu) (net 17) (status 80000))
   (segment (start 151.765 116.205) (end 151.7777 115.9891) (width 0.25) (layer F.Cu) (net 17) (status 80000))
-  (segment (start 137.16 122.428) (end 137.16 122.555) (width 0.25) (layer B.Cu) (net 18) (status 80000))
-  (segment (start 137.16 122.555) (end 134.62 119.38) (width 0.25) (layer B.Cu) (net 18) (status 80000))
+  (segment (start 134.62 119.38) (end 134.62 120.015) (width 0.25) (layer B.Cu) (net 18))
+  (segment (start 142.875 98.425) (end 142.875 100.965) (width 0.25) (layer F.Cu) (net 18) (status 80000))
+  (segment (start 142.24 101.6) (end 142.875 100.965) (width 0.25) (layer F.Cu) (net 18) (status 80000))
+  (segment (start 140.97 101.6) (end 142.24 101.6) (width 0.25) (layer F.Cu) (net 18) (status 80000))
+  (segment (start 140.335 101.6) (end 140.97 101.6) (width 0.25) (layer F.Cu) (net 18) (status 80000))
+  (segment (start 135.255 101.6) (end 140.335 101.6) (width 0.25) (layer F.Cu) (net 18) (status 80000))
+  (segment (start 134.62 102.235) (end 135.255 101.6) (width 0.25) (layer F.Cu) (net 18) (status 80000))
+  (segment (start 134.62 107.95) (end 134.62 102.235) (width 0.25) (layer F.Cu) (net 18) (status 80000))
+  (segment (start 134.62 118.745) (end 134.62 107.95) (width 0.25) (layer F.Cu) (net 18) (status 80000))
+  (segment (start 134.62 119.38) (end 134.62 118.745) (width 0.25) (layer F.Cu) (net 18) (status 80000))
   (via (at 134.62 119.38) (size 0.6) (layers F.Cu B.Cu) (net 18) (status 80000))
-  (segment (start 134.62 119.38) (end 134.62 118.745) (width 0.25) (layer F.Cu) (net 18) (status 80000))
-  (segment (start 134.62 118.745) (end 134.62 107.95) (width 0.25) (layer F.Cu) (net 18) (status 80000))
-  (segment (start 134.62 107.95) (end 134.62 102.235) (width 0.25) (layer F.Cu) (net 18) (status 80000))
-  (segment (start 134.62 102.235) (end 135.255 101.6) (width 0.25) (layer F.Cu) (net 18) (status 80000))
-  (segment (start 135.255 101.6) (end 140.335 101.6) (width 0.25) (layer F.Cu) (net 18) (status 80000))
-  (segment (start 140.335 101.6) (end 140.97 101.6) (width 0.25) (layer F.Cu) (net 18) (status 80000))
-  (segment (start 140.97 101.6) (end 142.24 101.6) (width 0.25) (layer F.Cu) (net 18) (status 80000))
-  (segment (start 142.24 101.6) (end 142.875 100.965) (width 0.25) (layer F.Cu) (net 18) (status 80000))
-  (segment (start 142.875 100.965) (end 142.875 98.425) (width 0.25) (layer F.Cu) (net 18) (status 80000))
+  (segment (start 135.89 121.285) (end 137.16 121.285) (width 0.25) (layer B.Cu) (net 18))
+  (segment (start 134.62 120.015) (end 135.89 121.285) (width 0.25) (layer B.Cu) (net 18))
   (segment (start 142.875 98.425) (end 142.748 98.552) (width 0.25) (layer F.Cu) (net 18) (status 80000))
 )
